File: motor_drivers.sch (KiCad schematic (older format))
At the start: 49 parts

Commit message: Added footprints.
Parts:
- C10, C12, C8: renamed from C?; footprint (none) -> Capacitor_SMD:C_0805_2012Metric
- C11, C13, C14, C15, C16, C17, C18, C19, C20, C21, C22, C23, C9: renamed from C?; footprint (none) -> Capacitor_SMD:C_0603_1608Metric
- D4, D5, D6, D7, D8, D9: renamed from D?; footprint (none) -> Diode_SMD:D_SMB_Handsoldering
- R10, R11, R12, R13, R14, R15, R16, R17, R18, R19, R20, R21, R4, R5, R6, R7, R8, R9: renamed from R?; footprint (none) -> Resistor_SMD:R_0603_1608Metric
- gave numbers to parts that had none: 9
