File: autophon-nerdblatt.kicad_pcb (KiCad board)
At the start: 2 copper layers, 265 x 50.6 mm, 98 parts, among them J1 Conn_01x06_Female, J101 board-edge-connector, J2 Conn_02x06_Odd_Even, Q300 BSS84, Q301 BSS84, Q302 BSS84, Q303 BSS84, Q304 BSS84, Q305 BSS84, SW1 SW_Push, SW2 SW_Push, U101 LM1117-3.3, U102 LM2594M-5.0, U201 SN74LV1T34, U202 SN74LV1T34, U203 74AHCT595, U204 SN74LV1T34, U205 74AHCT595, U206 ESP32-WROOM-32, U207 74AHCT595, U300 L298HN, U301 L298HN, U302 L298HN

Commit message: add Display sheet and I2C Pullups
Parts:
- added C1: 1u, Capacitor_SMD:C_0805_2012Metric, F.Cu at (111.0, 103.4)
- added C2: 1u, Capacitor_SMD:C_0805_2012Metric, F.Cu at (106.5, 103.4)
- added C3: 1u, Capacitor_SMD:C_0805_2012Metric, F.Cu at (102.1, 106.4)
- added C4: 100n, Capacitor_SMD:C_0603_1608Metric, F.Cu at (110.8, 106.1)
- added C5: 10u, Capacitor_SMD:C_0805_2012Metric, F.Cu at (106.5, 106.4)
- added C6: 10u, Capacitor_SMD:C_0805_2012Metric, F.Cu at (102.1, 103.4)
- added R4: 10k, Resistor_SMD:R_0603_1608Metric, F.Cu at (177.0, 120.1)
- added R5: 10k, Resistor_SMD:R_0603_1608Metric, F.Cu at (177.0, 124.2)
- added R6: 910k, Resistor_SMD:R_0603_1608Metric, F.Cu at (110.8, 108.6)
- added U1: EA_W096016-XALW, Display:EA W096016-XA, F.Cu at (86.9, 106.2)
- D201, D202, D300, D301, D302, D303, D304, D305: value 5v1 -> 5v6
Connections:
- J101 pad 12A: no_connect_95 -> no_connect_105
- J101 pad 13A: no_connect_96 -> no_connect_106
- J101 pad 14A: no_connect_97 -> no_connect_107
- J101 pad 15A: no_connect_98 -> no_connect_108
- J101 pad 15B: no_connect_99 -> no_connect_109
- J101 pad 16A: no_connect_100 -> no_connect_110
- J101 pad 16B: no_connect_101 -> no_connect_111
- J101 pad 17A: no_connect_102 -> no_connect_112
- J101 pad 18A: no_connect_103 -> no_connect_113
- J101 pad 19A: no_connect_104 -> no_connect_114
- J101 pad 1A: no_connect_105 -> no_connect_115
- J101 pad 1B: no_connect_106 -> no_connect_116
- J101 pad 20A: no_connect_107 -> no_connect_117
- J101 pad 21A: no_connect_108 -> no_connect_118
- J101 pad 21B: no_connect_109 -> no_connect_119
- J101 pad 22A: no_connect_110 -> no_connect_120
- J101 pad 22B: no_connect_111 -> no_connect_121
- J101 pad 23B: no_connect_112 -> no_connect_122
- J101 pad 24B: no_connect_113 -> no_connect_123
- J101 pad 25B: no_connect_114 -> no_connect_124
- J101 pad 26A: no_connect_115 -> no_connect_125
- J101 pad 26B: no_connect_116 -> no_connect_126
- J101 pad 27B: no_connect_117 -> no_connect_127
- J101 pad 28B: no_connect_118 -> no_connect_128
- J101 pad 29B: no_connect_119 -> no_connect_129
- J101 pad 2A: no_connect_120 -> no_connect_130
- J101 pad 2B: no_connect_121 -> no_connect_131
- J101 pad 30A: no_connect_122 -> no_connect_132
- J101 pad 30B: no_connect_123 -> no_connect_133
- J101 pad 31B: no_connect_124 -> no_connect_134
- J101 pad 32B: no_connect_125 -> no_connect_135
- J101 pad 33B: no_connect_126 -> no_connect_136
- J101 pad 34A: no_connect_127 -> no_connect_137
- J101 pad 36B: no_connect_128 -> no_connect_138
- J101 pad 38A: no_connect_129 -> no_connect_139
- J101 pad 38B: no_connect_130 -> no_connect_140
- J101 pad 39A: no_connect_131 -> no_connect_141
- J101 pad 3A: no_connect_132 -> no_connect_142
- J101 pad 3B: no_connect_133 -> no_connect_143
- J101 pad 40A: no_connect_134 -> no_connect_144
- J101 pad 40B: no_connect_135 -> no_connect_145
- J101 pad 41A: no_connect_136 -> no_connect_146
- J101 pad 41B: no_connect_137 -> no_connect_147
- J101 pad 42A: no_connect_138 -> no_connect_148
- J101 pad 42B: no_connect_139 -> no_connect_149
- J101 pad 43A: no_connect_140 -> no_connect_150
- J101 pad 43B: no_connect_141 -> no_connect_151
- J101 pad 44A: no_connect_142 -> no_connect_152
- J101 pad 44B: no_connect_143 -> no_connect_153
- J101 pad 4A: no_connect_144 -> no_connect_154
- J101 pad 4B: no_connect_145 -> no_connect_155
- J101 pad 5A: no_connect_146 -> no_connect_156
- J101 pad 5B: no_connect_147 -> no_connect_157
- J101 pad 6B: no_connect_148 -> no_connect_158
- J101 pad 7A: no_connect_149 -> no_connect_159
- J101 pad 7B: no_connect_150 -> no_connect_160
- J101 pad 8B: no_connect_151 -> no_connect_161
- J101 pad 9A: no_connect_152 -> no_connect_162
- U206 pad 17: no_connect_153 -> no_connect_163
- U206 pad 18: no_connect_154 -> no_connect_164
- U206 pad 19: no_connect_155 -> no_connect_165
- U206 pad 20: no_connect_156 -> no_connect_166
- U206 pad 21: no_connect_157 -> no_connect_167
- U206 pad 22: no_connect_158 -> no_connect_168
- U206 pad 24: no_connect_159 -> no_connect_169
- U206 pad 32: no_connect_160 -> (no net)
- U206 pad 4: no_connect_161 -> no_connect_170
- U206 pad 5: no_connect_162 -> no_connect_171
Routing:
- net /ESP32_Shiftregs/I2C_SDA: track 0.00 -> 1.21 mm

Commit message: Display Routing
Parts:
- moved R6 33.1 mm to (84.6, 88.4), turned to -90 degrees
- moved C4 32.9 mm to (83.1, 88.4), turned to 90 degrees
- moved C5 31.0 mm to (81.3, 88.4), turned to 90 degrees
- moved TP103 22.2 mm to (150.2, 113.3)
- moved C6 21.9 mm to (81.0, 97.3), turned to 90 degrees
- moved D103 19.6 mm to (155.7, 104.7)
- moved R103 19.6 mm to (155.7, 107.8)
- moved C1 18.7 mm to (93.2, 97.5), turned to 90 degrees
- moved C2 16.3 mm to (93.2, 94.0), turned to 90 degrees
- moved D102 14.1 mm to (144.2, 93.7), turned to 0 degrees
- moved U101 13.9 mm to (150.6, 107.1), turned to -90 degrees
- moved R102 12.6 mm to (144.2, 92.1), turned to 0 degrees
- moved C105 11.5 mm to (144.8, 106.5), turned to -90 degrees
- moved C106 11.3 mm to (153.6, 100.7), turned to 0 degrees
- moved C3 10.3 mm to (93.2, 101.1), turned to -90 degrees
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Connections:
- J101 pad 12A: no_connect_105 -> no_connect_103
- J101 pad 13A: no_connect_106 -> no_connect_104
- J101 pad 14A: no_connect_107 -> no_connect_105
- J101 pad 15A: no_connect_108 -> no_connect_106
- J101 pad 15B: no_connect_109 -> no_connect_107
- J101 pad 16A: no_connect_110 -> no_connect_108
- J101 pad 16B: no_connect_111 -> no_connect_109
- J101 pad 17A: no_connect_112 -> no_connect_110
- J101 pad 18A: no_connect_113 -> no_connect_111
- J101 pad 19A: no_connect_114 -> no_connect_112
- J101 pad 1A: no_connect_115 -> no_connect_113
- J101 pad 1B: no_connect_116 -> no_connect_114
- J101 pad 20A: no_connect_117 -> no_connect_115
- J101 pad 21A: no_connect_118 -> no_connect_116
- J101 pad 21B: no_connect_119 -> no_connect_117
- J101 pad 22A: no_connect_120 -> no_connect_118
- J101 pad 22B: no_connect_121 -> no_connect_119
- J101 pad 23B: no_connect_122 -> no_connect_120
- J101 pad 24B: no_connect_123 -> no_connect_121
- J101 pad 25B: no_connect_124 -> no_connect_122
- J101 pad 26A: no_connect_125 -> no_connect_123
- J101 pad 26B: no_connect_126 -> no_connect_124
- J101 pad 27B: no_connect_127 -> no_connect_125
- J101 pad 28B: no_connect_128 -> no_connect_126
- J101 pad 29B: no_connect_129 -> no_connect_127
- J101 pad 2A: no_connect_130 -> no_connect_128
- J101 pad 2B: no_connect_131 -> no_connect_129
- J101 pad 30A: no_connect_132 -> no_connect_130
- J101 pad 30B: no_connect_133 -> no_connect_131
- J101 pad 31B: no_connect_134 -> no_connect_132
- J101 pad 32B: no_connect_135 -> no_connect_133
- J101 pad 33B: no_connect_136 -> no_connect_134
- J101 pad 34A: no_connect_137 -> no_connect_135
- J101 pad 36B: no_connect_138 -> no_connect_136
- J101 pad 38A: no_connect_139 -> no_connect_137
- J101 pad 38B: no_connect_140 -> no_connect_138
- J101 pad 39A: no_connect_141 -> no_connect_139
- J101 pad 3A: no_connect_142 -> no_connect_140
- J101 pad 3B: no_connect_143 -> no_connect_141
- J101 pad 40A: no_connect_144 -> no_connect_142
- J101 pad 40B: no_connect_145 -> no_connect_143
- J101 pad 41A: no_connect_146 -> no_connect_144
- J101 pad 41B: no_connect_147 -> no_connect_145
- J101 pad 42A: no_connect_148 -> no_connect_146
- J101 pad 42B: no_connect_149 -> no_connect_147
- J101 pad 43A: no_connect_150 -> no_connect_148
- J101 pad 43B: no_connect_151 -> no_connect_149
- J101 pad 44A: no_connect_152 -> no_connect_150
- J101 pad 44B: no_connect_153 -> no_connect_151
- J101 pad 4A: no_connect_154 -> no_connect_152
- J101 pad 4B: no_connect_155 -> no_connect_153
- J101 pad 5A: no_connect_156 -> no_connect_154
- J101 pad 5B: no_connect_157 -> no_connect_155
- J101 pad 6B: no_connect_158 -> no_connect_156
- J101 pad 7A: no_connect_159 -> no_connect_157
- J101 pad 7B: no_connect_160 -> no_connect_158
- J101 pad 8B: no_connect_161 -> no_connect_159
- J101 pad 9A: no_connect_162 -> no_connect_160
- R4 pad 2: /ESP32_Shiftregs/I2C_SDA -> I2C_SDA
- R5 pad 2: /ESP32_Shiftregs/I2C_SCL -> I2C_SCL
- U206 pad 17: no_connect_163 -> no_connect_161
- U206 pad 18: no_connect_164 -> no_connect_162
- U206 pad 19: no_connect_165 -> no_connect_163
- U206 pad 20: no_connect_166 -> no_connect_164
- U206 pad 21: no_connect_167 -> no_connect_165
- U206 pad 22: no_connect_168 -> no_connect_166
- U206 pad 24: no_connect_169 -> no_connect_167
- U206 pad 33: /ESP32_Shiftregs/I2C_SDA -> I2C_SDA
- U206 pad 36: /ESP32_Shiftregs/I2C_SCL -> I2C_SCL
- U206 pad 4: no_connect_170 -> no_connect_168
- U206 pad 5: no_connect_171 -> no_connect_169
Routing:
- net I2C_SCL: track 0.00 -> 119.6 mm, vias 0 -> 2
- net I2C_SDA: track 0.00 -> 117.4 mm
- net VCC: track 253.1 -> 338.8 mm
- net Net-(U1-Pad13): track 0.00 -> 11.1 mm
- net Net-(U1-Pad12): track 0.00 -> 9.16 mm
- net Net-(U1-Pad4): track 0.00 -> 8.95 mm
- net +24V: track 264.3 -> 256.4 mm
- net Net-(U1-Pad3): track 0.00 -> 6.50 mm
- net ABCDEF_HALL_GND: track 23.0 -> 16.6 mm, vias 55 -> 22
- net Net-(U1-Pad2): track 0.00 -> 4.66 mm
- net Net-(U1-Pad1): track 0.00 -> 2.45 mm
- net /ESP32_Shiftregs/~HALL_EN_3V~: track 61.2 -> 63.2 mm
- net +5V: track 343.1 -> 345.1 mm
- net Net-(U1-Pad14): track 0.00 -> 1.84 mm
- net Net-(Q305-Pad2): track 1.65 -> 3.30 mm
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
Commit message: Layout cleanup
Parts:
- moved R3 16.9 mm to (228.0, 105.3), turned to -90 degrees
Routing:
- net VCC: track 338.8 -> 312.5 mm, vias 6 -> 9
- net /ESP32_Shiftregs/HALL_INDEX_3V: track 84.4 -> 89.1 mm
- net /ESP32_Shiftregs/SPI_CLK: track 114.7 -> 112.0 mm
- net /ESP32_Shiftregs/~HALL_EN_3V~: track 63.2 -> 65.9 mm
- net +5V: track 345.1 -> 342.9 mm
- net /ESP32_Shiftregs/ESP32_GPIO0: track 35.0 -> 33.2 mm
- net /ESP32_Shiftregs/SPI_COPI: track 88.7 -> 90.3 mm, vias 3 -> 4
- net /ESP32_Shiftregs/HALL_ROTOR_3V: track 80.5 -> 79.2 mm
- net /ESP32_Shiftregs/~SPI_CSO~: track 127.2 -> 128.3 mm, vias 7 -> 6
- net Net-(U203-Pad9): track 34.8 -> 33.9 mm
- net A_MOT_NEG_DRV: track 51.1 -> 50.1 mm
- net /ESP32_Shiftregs/MOT_EN_3V: track 72.6 -> 73.4 mm
- net B_MOT_POS_DRV: track 56.6 -> 55.9 mm
- net C_MOT_NEG_DRV: track 29.7 -> 29.0 mm
- net I2C_SCL: track 119.6 -> 119.0 mm
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
Commit message: GND Vias and Bus Resistors in series.
Parts:
- added R10: 33R, Resistor_SMD:R_0603_1608Metric, F.Cu at (177.2, 120.3)
- added R11: 33R, Resistor_SMD:R_0603_1608Metric, F.Cu at (177.2, 124.2)
- added R12: 33R, Resistor_SMD:R_0603_1608Metric, F.Cu at (263.9, 114.3)
- added R13: 33R, Resistor_SMD:R_0603_1608Metric, F.Cu at (286.7, 114.7)
- added R7: 33R, Resistor_SMD:R_0603_1608Metric, F.Cu at (193.9, 107.1)
- added R8: 33R, Resistor_SMD:R_0603_1608Metric, F.Cu at (199.9, 111.4)
- added R9: 33R, Resistor_SMD:R_0603_1608Metric, F.Cu at (185.0, 106.9)
- moved R3 11.4 mm to (216.6, 106.2), turned to 180 degrees
- moved R5 1.47 mm to (177.2, 125.7), turned to 180 degrees
- moved R4 1.40 mm to (177.2, 118.8), turned to 180 degrees
- moved C107 0.89 mm to (203.4, 120.8)
Connections:
- J101 pad 12A: no_connect_103 -> no_connect_112
- J101 pad 13A: no_connect_104 -> no_connect_113
- J101 pad 14A: no_connect_105 -> no_connect_114
- J101 pad 15A: no_connect_106 -> no_connect_115
- J101 pad 15B: no_connect_107 -> no_connect_116
- J101 pad 16A: no_connect_108 -> no_connect_117
- J101 pad 16B: no_connect_109 -> no_connect_118
- J101 pad 17A: no_connect_110 -> no_connect_119
- J101 pad 18A: no_connect_111 -> no_connect_120
- J101 pad 19A: no_connect_112 -> no_connect_121
- J101 pad 1A: no_connect_113 -> no_connect_122
- J101 pad 1B: no_connect_114 -> no_connect_123
- J101 pad 20A: no_connect_115 -> no_connect_124
- J101 pad 21A: no_connect_116 -> no_connect_125
- J101 pad 21B: no_connect_117 -> no_connect_126
- J101 pad 22A: no_connect_118 -> no_connect_127
- J101 pad 22B: no_connect_119 -> no_connect_128
- J101 pad 23B: no_connect_120 -> no_connect_129
- J101 pad 24B: no_connect_121 -> no_connect_130
- J101 pad 25B: no_connect_122 -> no_connect_131
- J101 pad 26A: no_connect_123 -> no_connect_132
- J101 pad 26B: no_connect_124 -> no_connect_133
- J101 pad 27B: no_connect_125 -> no_connect_134
- J101 pad 28B: no_connect_126 -> no_connect_135
- J101 pad 29B: no_connect_127 -> no_connect_136
- J101 pad 2A: no_connect_128 -> no_connect_137
- J101 pad 2B: no_connect_129 -> no_connect_138
- J101 pad 30A: no_connect_130 -> no_connect_139
- J101 pad 30B: no_connect_131 -> no_connect_140
- J101 pad 31B: no_connect_132 -> no_connect_141
- J101 pad 32B: no_connect_133 -> no_connect_142
- J101 pad 33B: no_connect_134 -> no_connect_143
- J101 pad 34A: no_connect_135 -> no_connect_144
- J101 pad 36B: no_connect_136 -> no_connect_145
- J101 pad 38A: no_connect_137 -> no_connect_146
- J101 pad 38B: no_connect_138 -> no_connect_147
- J101 pad 39A: no_connect_139 -> no_connect_148
- J101 pad 3A: no_connect_140 -> no_connect_149
- J101 pad 3B: no_connect_141 -> no_connect_150
- J101 pad 40A: no_connect_142 -> no_connect_151
- J101 pad 40B: no_connect_143 -> no_connect_152
- J101 pad 41A: no_connect_144 -> no_connect_153
- J101 pad 41B: no_connect_145 -> no_connect_154
- J101 pad 42A: no_connect_146 -> no_connect_155
- J101 pad 42B: no_connect_147 -> no_connect_156
- J101 pad 43A: no_connect_148 -> no_connect_157
- J101 pad 43B: no_connect_149 -> no_connect_158
- J101 pad 44A: no_connect_150 -> no_connect_159
- J101 pad 44B: no_connect_151 -> no_connect_160
- J101 pad 4A: no_connect_152 -> no_connect_161
- J101 pad 4B: no_connect_153 -> no_connect_162
- J101 pad 5A: no_connect_154 -> no_connect_163
- J101 pad 5B: no_connect_155 -> no_connect_164
- J101 pad 6B: no_connect_156 -> no_connect_165
- J101 pad 7A: no_connect_157 -> no_connect_166
- J101 pad 7B: no_connect_158 -> no_connect_167
- J101 pad 8B: no_connect_159 -> no_connect_168
- J101 pad 9A: no_connect_160 -> no_connect_169
- J2 pad 2: /ESP32_Shiftregs/SPI_COPI -> /ESP32_Shiftregs/SPI_COPI-t
- J2 pad 3: /ESP32_Shiftregs/SPI_CLK -> /ESP32_Shiftregs/SPI_CLK-t
- J2 pad 4: /ESP32_Shiftregs/~SPI_CSO~ -> /ESP32_Shiftregs/~SPI_CSO-t~
- R3 pad 2: /ESP32_Shiftregs/~SPI_CSO~ -> /ESP32_Shiftregs/~SPI_CSO-t~
- R4 pad 2: I2C_SDA -> I2C_SDA-t
- R5 pad 2: I2C_SCL -> I2C_SCL-t
- U203 pad 11: /ESP32_Shiftregs/SPI_CLK -> /ESP32_Shiftregs/SPI_CLK-t
- U203 pad 12: /ESP32_Shiftregs/~SPI_CSO~ -> /ESP32_Shiftregs/~SPI_CSO-t~
- U203 pad 14: /ESP32_Shiftregs/SPI_COPI -> /ESP32_Shiftregs/SPI_COPI-t
- U203 pad 9: Net-(U203-Pad9) -> Net-(R12-Pad1)
- U205 pad 11: /ESP32_Shiftregs/SPI_CLK -> /ESP32_Shiftregs/SPI_CLK-t
- U205 pad 12: /ESP32_Shiftregs/~SPI_CSO~ -> /ESP32_Shiftregs/~SPI_CSO-t~
- U205 pad 14: Net-(U203-Pad9) -> Net-(R12-Pad2)
- U205 pad 9: Net-(U205-Pad9) -> Net-(R13-Pad1)
- U206 pad 17: no_connect_161 -> no_connect_170
- U206 pad 18: no_connect_162 -> no_connect_171
- U206 pad 19: no_connect_163 -> no_connect_172
- U206 pad 20: no_connect_164 -> no_connect_173
- U206 pad 21: no_connect_165 -> no_connect_174
- U206 pad 22: no_connect_166 -> no_connect_175
- U206 pad 24: no_connect_167 -> no_connect_176
- U206 pad 33: I2C_SDA -> /ESP32_Shiftregs/I2C_SDA
- U206 pad 36: I2C_SCL -> /ESP32_Shiftregs/I2C_SCL
- U206 pad 4: no_connect_168 -> no_connect_177
- U206 pad 5: no_connect_169 -> no_connect_178
- U207 pad 11: /ESP32_Shiftregs/SPI_CLK -> /ESP32_Shiftregs/SPI_CLK-t
- U207 pad 12: /ESP32_Shiftregs/~SPI_CSO~ -> /ESP32_Shiftregs/~SPI_CSO-t~
- U207 pad 14: Net-(U205-Pad9) -> /ESP32_Shiftregs/SER_QH_2
Routing:
- net /ESP32_Shiftregs/~SPI_CSO-t~: track 0.00 -> 130.5 mm, vias 0 -> 6
- net /ESP32_Shiftregs/~SPI_CSO~: track 128.3 -> 2.23 mm, vias 6 -> 0
- net I2C_SCL: track 119.0 -> 0.00 mm, vias 2 -> 0
- net I2C_SCL-t: track 0.00 -> 117.5 mm, vias 0 -> 2
- net I2C_SDA: track 117.2 -> 0.00 mm, vias 2 -> 0
- net I2C_SDA-t: track 0.00 -> 114.5 mm, vias 0 -> 2
- net /ESP32_Shiftregs/SPI_CLK-t: track 0.00 -> 111.7 mm, vias 0 -> 6
- net /ESP32_Shiftregs/SPI_CLK: track 112.0 -> 2.03 mm, vias 6 -> 0
- net /ESP32_Shiftregs/SPI_COPI-t: track 0.00 -> 88.8 mm, vias 0 -> 4
- net /ESP32_Shiftregs/SPI_COPI: track 90.3 -> 2.06 mm, vias 4 -> 0
- net Net-(U205-Pad9): track 87.0 -> 0.00 mm, vias 4 -> 0
- net /ESP32_Shiftregs/SER_QH_2: track 0.00 -> 83.6 mm, vias 0 -> 4
- net Net-(R12-Pad2): track 0.00 -> 37.2 mm, vias 0 -> 2
- net Net-(U203-Pad9): track 33.9 -> 0.00 mm, vias 2 -> 0
- net +5V: track 342.9 -> 365.9 mm, vias 11 -> 12
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
Commit message: Logo, fun and cleanup
Parts:
- added G***: LOGO, Grafiks:nerdberglogo, F.Cu at (99.0, 84.3)
Routing:
- net ABCDEF_HALL_GND: vias 2201 -> 2219
Other:
- board text added: ""Flip flap flupperdupperdob Flupperdupperblib og flop" Pilfingerdansen - Sigurd Barrett"
