File: autophon-nerdblatt.kicad_sch (KiCad schematic)
At the start: 21 parts, among them J101 board-edge-connector, U101 LM1117-3.3, U102 LM2594M-5.0

Commit message: add Display sheet and I2C Pullups
Parts:
- C104: Link https://www.reichelt.de/smd-vielschicht-keramikkondensator-100n-10--x7r-g0603-100n-p31873.html?&trstct=pos_1&nbc=1 -> https://www.reichelt.de/smd-vielschicht-keramikkondensator-100n-10--x7r-g0603-100n-p31873.html?&trstct=pos_3&nbc=1
Other:
- added sheet Display_Sensors (display_sens.kicad_sch)
