File: display_sens.kicad_sch (KiCad schematic)
At the start: 8 parts, among them U1 EA_W096016-XALW

Commit message: BOM
Parts:
- R6: Distri (none) -> Reichelt; Link (none) -> https://www.reichelt.de/smd-widerstand-0603-910-kohm-100-mw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
Changed lines of the file:
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@@
+      (effects (font (size 1.27 1.27)) hide)
+    )
+    (property "Distri" "Reichelt" (id 4) (at 41.91 67.31 0)
+      (effects (font (size 1.27 1.27)) hide)
+    )
+    (property "Link" "https://www.reichelt.de/smd-widerstand-0603-910-kohm-100-mw-1--rnd-0603-1-910k-p183123.html?search=0603+910" (id 5) (at 41.91 67.31 0)
       (effects (font (size 1.27 1.27)) hide)
     )
