File: motor_drivers.kicad_sch (KiCad schematic)
At the start: 48 parts, among them Q300 BSS84, Q301 BSS84, Q302 BSS84, Q303 BSS84, Q304 BSS84, Q305 BSS84, U300 L298HN, U301 L298HN, U302 L298HN

Commit message: more C vor Logic and placing first groups of parts
Parts:
- D300, D301, D302, D303, D304, D305: footprint Diode_SMD:D_SMB_Handsoldering -> Diode_SMD:D_SOT-23_ANK; Link https://www.reichelt.de/zenerdiode-5-1-v-3-w-smb-1smb-5918b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 -> https://www.reichelt.de/zenerdiode-5-1-v-0-35-w-sot-23-smd-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
Changed lines of the file:
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@@
       (effects (font (size 1.27 1.27)) (justify left))
     )
-    (property "Footprint" "Diode_SMD:D_SMB_Handsoldering" (id 2) (at 252.73 26.67 0)
+    (property "Footprint" "Diode_SMD:D_SOT-23_ANK" (id 2) (at 252.73 26.67 0)
       (effects (font (size 1.27 1.27)) hide)
     )
@@
       (effects (font (size 1.27 1.27)) hide)
     )
-    (property "Link" "https://www.reichelt.de/zenerdiode-5-1-v-3-w-smb-1smb-5918bt3g-p219392.html?search=Zenerdiode%2C+5%2C1+V" (id 5) (at 252.73 26.67 0)
+    (property "Link" "https://www.reichelt.de/zenerdiode-5-1-v-0-35-w-sot-23-smd-zd-5-1-p18916.html?&trstct=pos_3&nbc=1" (id 5) (at 252.73 26.67 0)
       (effects (font (size 1.27 1.27)) hide)
     )
@@
       (effects (font (size 1.27 1.27)) (justify left))
     )
-    (property "Footprint" "Diode_SMD:D_SMB_Handsoldering" (id 2) (at 252.73 52.07 0)
+    (property "Footprint" "Diode_SMD:D_SOT-23_ANK" (id 2) (at 252.73 52.07 0)
       (effects (font (size 1.27 1.27)) hide)
     )
@@
       (effects (font (size 1.27 1.27)) hide)
     )
-    (property "Link" "https://www.reichelt.de/zenerdiode-5-1-v-3-w-smb-1smb-5918bt3g-p219392.html?search=Zenerdiode%2C+5%2C1+V" (id 5) (at 252.73 52.07 0)
+    (property "Link" "https://www.reichelt.de/zenerdiode-5-1-v-0-35-w-sot-23-smd-zd-5-1-p18916.html?&trstct=pos_3&nbc=1" (id 5) (at 252.73 52.07 0)
       (effects (font (size 1.27 1.27)) hide)
     )
@@
       (effects (font (size 1.27 1.27)) (justify left))
     )
-    (property "Footprint" "Diode_SMD:D_SMB_Handsoldering" (id 2) (at 252.73 77.47 0)
+    (property "Footprint" "Diode_SMD:D_SOT-23_ANK" (id 2) (at 252.73 77.47 0)
       (effects (font (size 1.27 1.27)) hide)
     )
@@
       (effects (font (size 1.27 1.27)) hide)
     )
-    (property "Link" "https://www.reichelt.de/zenerdiode-5-1-v-3-w-smb-1smb-5918bt3g-p219392.html?search=Zenerdiode%2C+5%2C1+V" (id 5) (at 252.73 77.47 0)
+    (property "Link" "https://www.reichelt.de/zenerdiode-5-1-v-0-35-w-sot-23-smd-zd-5-1-p18916.html?&trstct=pos_3&nbc=1" (id 5) (at 252.73 77.47 0)
       (effects (font (size 1.27 1.27)) hide)
     )
@@
       (effects (font (size 1.27 1.27)) (justify left))
     )
-    (property "Footprint" "Diode_SMD:D_SMB_Handsoldering" (id 2) (at 252.73 102.87 0)
+    (property "Footprint" "Diode_SMD:D_SOT-23_ANK" (id 2) (at 252.73 102.87 0)
       (effects (font (size 1.27 1.27)) hide)
     )
@@
       (effects (font (size 1.27 1.27)) hide)
     )
-    (property "Link" "https://www.reichelt.de/zenerdiode-5-1-v-3-w-smb-1smb-5918bt3g-p219392.html?search=Zenerdiode%2C+5%2C1+V" (id 5) (at 252.73 102.87 0)
+    (property "Link" "https://www.reichelt.de/zenerdiode-5-1-v-0-35-w-sot-23-smd-zd-5-1-p18916.html?&trstct=pos_3&nbc=1" (id 5) (at 252.73 102.87 0)
       (effects (font (size 1.27 1.27)) hide)
     )
@@
       (effects (font (size 1.27 1.27)) (justify left))
     )
-    (property "Footprint" "Diode_SMD:D_SMB_Handsoldering" (id 2) (at 252.73 128.27 0)
+    (property "Footprint" "Diode_SMD:D_SOT-23_ANK" (id 2) (at 252.73 128.27 0)
       (effects (font (size 1.27 1.27)) hide)
     )
@@
       (effects (font (size 1.27 1.27)) hide)
     )
-    (property "Link" "https://www.reichelt.de/zenerdiode-5-1-v-3-w-smb-1smb-5918bt3g-p219392.html?search=Zenerdiode%2C+5%2C1+V" (id 5) (at 252.73 128.27 0)
+    (property "Link" "https://www.reichelt.de/zenerdiode-5-1-v-0-35-w-sot-23-smd-zd-5-1-p18916.html?&trstct=pos_3&nbc=1" (id 5) (at 252.73 128.27 0)
       (effects (font (size 1.27 1.27)) hide)
     )
@@
       (effects (font (size 1.27 1.27)) (justify left))
     )
-    (property "Footprint" "Diode_SMD:D_SMB_Handsoldering" (id 2) (at 252.73 153.67 0)
+    (property "Footprint" "Diode_SMD:D_SOT-23_ANK" (id 2) (at 252.73 153.67 0)
       (effects (font (size 1.27 1.27)) hide)
     )
@@
       (effects (font (size 1.27 1.27)) hide)
     )
-    (property "Link" "https://www.reichelt.de/zenerdiode-5-1-v-3-w-smb-1smb-5918bt3g-p219392.html?search=Zenerdiode%2C+5%2C1+V" (id 5) (at 252.73 153.67 0)
+    (property "Link" "https://www.reichelt.de/zenerdiode-5-1-v-0-35-w-sot-23-smd-zd-5-1-p18916.html?&trstct=pos_3&nbc=1" (id 5) (at 252.73 153.67 0)
       (effects (font (size 1.27 1.27)) hide)
     )

Commit message: all traces routed. ready for cleanup
Parts:
- U300, U301, U302: Distri (none) -> Reichelt; Link (none) -> https://www.reichelt.de/doppelvollbrueckentreiber-multiwatt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
Changed lines of the file:
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@@
+      (effects (font (size 1.27 1.27)) hide)
+    )
+    (property "Distri" "Reichelt" (id 4) (at 73.66 36.83 0)
+      (effects (font (size 1.27 1.27)) hide)
+    )
+    (property "Link" "https://www.reichelt.de/doppelvollbrueckentreiber-multiwatt-15-l-298-p9667.html?search=L298" (id 5) (at 73.66 36.83 0)
       (effects (font (size 1.27 1.27)) hide)
     )
@@
       (effects (font (size 1.27 1.27)) hide)
     )
+    (property "Distri" "Reichelt" (id 4) (at 73.66 85.09 0)
+      (effects (font (size 1.27 1.27)) hide)
+    )
+    (property "Link" "https://www.reichelt.de/doppelvollbrueckentreiber-multiwatt-15-l-298-p9667.html?search=L298" (id 5) (at 73.66 85.09 0)
+      (effects (font (size 1.27 1.27)) hide)
+    )
   )
   (symbol (lib_id "Driver_Motor:L298HN") (at 73.66 133.35 0) (unit 1)
@@
       (effects (font (size 1.27 1.27)) hide)
     )
+    (property "Distri" "Reichelt" (id 4) (at 73.66 133.35 0)
+      (effects (font (size 1.27 1.27)) hide)
+    )
+    (property "Link" "https://www.reichelt.de/doppelvollbrueckentreiber-multiwatt-15-l-298-p9667.html?search=L298" (id 5) (at 73.66 133.35 0)
+      (effects (font (size 1.27 1.27)) hide)
+    )

Commit message: Zener diodes now 5v6
Parts:
- D300, D301, D302, D303, D304, D305: value 5v1 -> 5v6; Link https://www.reichelt.de/zenerdiode-5-1-v-0-35-w-sot-23-smd-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 -> https://www.reichelt.de/zenerdiode-5-6-v-0-35-w-sot-23-smd-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
Changed lines of the file:
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@@
       (effects (font (size 1.27 1.27)) (justify left))
     )
-    (property "Value" "5v1" (id 1) (at 254.762 27.813 90)
+    (property "Value" "5v6" (id 1) (at 254.762 27.813 90)
       (effects (font (size 1.27 1.27)) (justify left))
     )
@@
       (effects (font (size 1.27 1.27)) hide)
     )
-    (property "Link" "https://www.reichelt.de/zenerdiode-5-1-v-0-35-w-sot-23-smd-zd-5-1-p18916.html?&trstct=pos_3&nbc=1" (id 5) (at 252.73 26.67 0)
+    (property "Link" "https://www.reichelt.de/zenerdiode-5-6-v-0-35-w-sot-23-smd-zd-5-6-p18917.html?&trstct=pos_0&nbc=1" (id 5) (at 252.73 26.67 0)
       (effects (font (size 1.27 1.27)) hide)
     )
@@
       (effects (font (size 1.27 1.27)) (justify left))
     )
-    (property "Value" "5v1" (id 1) (at 254.762 53.213 90)
+    (property "Value" "5v6" (id 1) (at 254.762 53.213 90)
       (effects (font (size 1.27 1.27)) (justify left))
     )
@@
       (effects (font (size 1.27 1.27)) hide)
     )
-    (property "Link" "https://www.reichelt.de/zenerdiode-5-1-v-0-35-w-sot-23-smd-zd-5-1-p18916.html?&trstct=pos_3&nbc=1" (id 5) (at 252.73 52.07 0)
+    (property "Link" "https://www.reichelt.de/zenerdiode-5-6-v-0-35-w-sot-23-smd-zd-5-6-p18917.html?&trstct=pos_0&nbc=1" (id 5) (at 252.73 52.07 0)
       (effects (font (size 1.27 1.27)) hide)
     )
@@
       (effects (font (size 1.27 1.27)) (justify left))
     )
-    (property "Value" "5v1" (id 1) (at 254.762 78.613 90)
+    (property "Value" "5v6" (id 1) (at 254.762 78.613 90)
       (effects (font (size 1.27 1.27)) (justify left))
     )
@@
       (effects (font (size 1.27 1.27)) hide)
     )
-    (property "Link" "https://www.reichelt.de/zenerdiode-5-1-v-0-35-w-sot-23-smd-zd-5-1-p18916.html?&trstct=pos_3&nbc=1" (id 5) (at 252.73 77.47 0)
+    (property "Link" "https://www.reichelt.de/zenerdiode-5-6-v-0-35-w-sot-23-smd-zd-5-6-p18917.html?&trstct=pos_0&nbc=1" (id 5) (at 252.73 77.47 0)
       (effects (font (size 1.27 1.27)) hide)
     )
@@
       (effects (font (size 1.27 1.27)) (justify left))
     )
-    (property "Value" "5v1" (id 1) (at 254.762 104.013 90)
+    (property "Value" "5v6" (id 1) (at 254.762 104.013 90)
       (effects (font (size 1.27 1.27)) (justify left))
     )
@@
       (effects (font (size 1.27 1.27)) hide)
     )
-    (property "Link" "https://www.reichelt.de/zenerdiode-5-1-v-0-35-w-sot-23-smd-zd-5-1-p18916.html?&trstct=pos_3&nbc=1" (id 5) (at 252.73 102.87 0)
+    (property "Link" "https://www.reichelt.de/zenerdiode-5-6-v-0-35-w-sot-23-smd-zd-5-6-p18917.html?&trstct=pos_0&nbc=1" (id 5) (at 252.73 102.87 0)
       (effects (font (size 1.27 1.27)) hide)
     )
@@
       (effects (font (size 1.27 1.27)) (justify left))
     )
-    (property "Value" "5v1" (id 1) (at 254.762 129.413 90)
+    (property "Value" "5v6" (id 1) (at 254.762 129.413 90)
       (effects (font (size 1.27 1.27)) (justify left))
     )
@@
       (effects (font (size 1.27 1.27)) hide)
     )
-    (property "Link" "https://www.reichelt.de/zenerdiode-5-1-v-0-35-w-sot-23-smd-zd-5-1-p18916.html?&trstct=pos_3&nbc=1" (id 5) (at 252.73 128.27 0)
+    (property "Link" "https://www.reichelt.de/zenerdiode-5-6-v-0-35-w-sot-23-smd-zd-5-6-p18917.html?&trstct=pos_0&nbc=1" (id 5) (at 252.73 128.27 0)
       (effects (font (size 1.27 1.27)) hide)
     )
@@
       (effects (font (size 1.27 1.27)) (justify left))
     )
-    (property "Value" "5v1" (id 1) (at 254.762 154.813 90)
+    (property "Value" "5v6" (id 1) (at 254.762 154.813 90)
       (effects (font (size 1.27 1.27)) (justify left))
     )
@@
       (effects (font (size 1.27 1.27)) hide)
     )
-    (property "Link" "https://www.reichelt.de/zenerdiode-5-1-v-0-35-w-sot-23-smd-zd-5-1-p18916.html?&trstct=pos_3&nbc=1" (id 5) (at 252.73 153.67 0)
+    (property "Link" "https://www.reichelt.de/zenerdiode-5-6-v-0-35-w-sot-23-smd-zd-5-6-p18917.html?&trstct=pos_0&nbc=1" (id 5) (at 252.73 153.67 0)
       (effects (font (size 1.27 1.27)) hide)
     )

Commit message: add Display sheet and I2C Pullups
Parts:
- C300, C301, C302, C303, C304, C305, C309, C311, C312: Link https://www.reichelt.de/smd-vielschicht-keramikkondensator-100n-10--x7r-g0603-100n-p31873.html?&trstct=pos_1&nbc=1 -> https://www.reichelt.de/smd-vielschicht-keramikkondensator-100n-10--x7r-g0603-100n-p31873.html?&trstct=pos_3&nbc=1
Changed lines of the file:
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@@
       (effects (font (size 1.27 1.27)) hide)
     )
-    (property "Link" "https://www.reichelt.de/smd-vielschicht-keramikkondensator-100n-10--x7r-g0603-100n-p31873.html?&trstct=pos_1&nbc=1" (id 5) (at 67.31 170.18 0)
+    (property "Link" "https://www.reichelt.de/smd-vielschicht-keramikkondensator-100n-10--x7r-g0603-100n-p31873.html?&trstct=pos_3&nbc=1" (id 5) (at 67.31 170.18 0)
       (effects (font (size 1.27 1.27)) hide)
     )
@@
       (effects (font (size 1.27 1.27)) hide)
     )
-    (property "Link" "https://www.reichelt.de/smd-vielschicht-keramikkondensator-100n-10--x7r-g0603-100n-p31873.html?&trstct=pos_1&nbc=1" (id 5) (at 80.01 170.18 0)
+    (property "Link" "https://www.reichelt.de/smd-vielschicht-keramikkondensator-100n-10--x7r-g0603-100n-p31873.html?&trstct=pos_3&nbc=1" (id 5) (at 80.01 170.18 0)
       (effects (font (size 1.27 1.27)) hide)
     )
@@
       (effects (font (size 1.27 1.27)) hide)
     )
-    (property "Link" "https://www.reichelt.de/smd-vielschicht-keramikkondensator-100n-10--x7r-g0603-100n-p31873.html?&trstct=pos_1&nbc=1" (id 5) (at 91.44 170.18 0)
+    (property "Link" "https://www.reichelt.de/smd-vielschicht-keramikkondensator-100n-10--x7r-g0603-100n-p31873.html?&trstct=pos_3&nbc=1" (id 5) (at 91.44 170.18 0)
       (effects (font (size 1.27 1.27)) hide)
     )
@@
       (effects (font (size 1.27 1.27)) hide)
     )
-    (property "Link" "https://www.reichelt.de/smd-vielschicht-keramikkondensator-100n-10--x7r-g0603-100n-p31873.html?&trstct=pos_1&nbc=1" (id 5) (at 243.84 26.67 0)
+    (property "Link" "https://www.reichelt.de/smd-vielschicht-keramikkondensator-100n-10--x7r-g0603-100n-p31873.html?&trstct=pos_3&nbc=1" (id 5) (at 243.84 26.67 0)
       (effects (font (size 1.27 1.27)) hide)
     )
@@
       (effects (font (size 1.27 1.27)) hide)
     )
-    (property "Link" "https://www.reichelt.de/smd-vielschicht-keramikkondensator-100n-10--x7r-g0603-100n-p31873.html?&trstct=pos_1&nbc=1" (id 5) (at 243.84 52.07 0)
+    (property "Link" "https://www.reichelt.de/smd-vielschicht-keramikkondensator-100n-10--x7r-g0603-100n-p31873.html?&trstct=pos_3&nbc=1" (id 5) (at 243.84 52.07 0)
       (effects (font (size 1.27 1.27)) hide)
     )
@@
       (effects (font (size 1.27 1.27)) hide)
     )
-    (property "Link" "https://www.reichelt.de/smd-vielschicht-keramikkondensator-100n-10--x7r-g0603-100n-p31873.html?&trstct=pos_1&nbc=1" (id 5) (at 243.84 77.47 0)
+    (property "Link" "https://www.reichelt.de/smd-vielschicht-keramikkondensator-100n-10--x7r-g0603-100n-p31873.html?&trstct=pos_3&nbc=1" (id 5) (at 243.84 77.47 0)
       (effects (font (size 1.27 1.27)) hide)
     )
@@
       (effects (font (size 1.27 1.27)) hide)
     )
-    (property "Link" "https://www.reichelt.de/smd-vielschicht-keramikkondensator-100n-10--x7r-g0603-100n-p31873.html?&trstct=pos_1&nbc=1" (id 5) (at 243.84 102.87 0)
+    (property "Link" "https://www.reichelt.de/smd-vielschicht-keramikkondensator-100n-10--x7r-g0603-100n-p31873.html?&trstct=pos_3&nbc=1" (id 5) (at 243.84 102.87 0)
       (effects (font (size 1.27 1.27)) hide)
     )
@@
       (effects (font (size 1.27 1.27)) hide)
     )
-    (property "Link" "https://www.reichelt.de/smd-vielschicht-keramikkondensator-100n-10--x7r-g0603-100n-p31873.html?&trstct=pos_1&nbc=1" (id 5) (at 243.84 128.27 0)
+    (property "Link" "https://www.reichelt.de/smd-vielschicht-keramikkondensator-100n-10--x7r-g0603-100n-p31873.html?&trstct=pos_3&nbc=1" (id 5) (at 243.84 128.27 0)
       (effects (font (size 1.27 1.27)) hide)
     )
@@
       (effects (font (size 1.27 1.27)) hide)
     )
-    (property "Link" "https://www.reichelt.de/smd-vielschicht-keramikkondensator-100n-10--x7r-g0603-100n-p31873.html?&trstct=pos_1&nbc=1" (id 5) (at 243.84 153.67 0)
+    (property "Link" "https://www.reichelt.de/smd-vielschicht-keramikkondensator-100n-10--x7r-g0603-100n-p31873.html?&trstct=pos_3&nbc=1" (id 5) (at 243.84 153.67 0)
       (effects (font (size 1.27 1.27)) hide)
     )

Commit message: BOM
Parts:
- R300, R303, R306, R309, R312, R315: Distri (none) -> Reichelt; Link (none) -> https://www.reichelt.de/smd-widerstand-0603-51-ohm-100-mw-1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
- R301, R302, R304, R305, R307, R308, R310, R311, R313, R314, R316, R317: Distri (none) -> Reichelt; Link (none) -> https://www.reichelt.de/smd-widerstand-0603-10-kohm-100-mw-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
Changed lines of the file:
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@@
+      (effects (font (size 1.27 1.27)) hide)
+    )
+    (property "Distri" "Reichelt" (id 4) (at 219.71 26.67 0)
+      (effects (font (size 1.27 1.27)) hide)
+    )
+    (property "Link" "https://www.reichelt.de/smd-widerstand-0603-10-kohm-100-mw-1--rnd-0603-1-10k-p183077.html?search=10k+0603" (id 5) (at 219.71 26.67 0)
       (effects (font (size 1.27 1.27)) hide)
     )
@@
       (effects (font (size 1.27 1.27)) hide)
     )
+    (property "Distri" "Reichelt" (id 4) (at 219.71 52.07 0)
+      (effects (font (size 1.27 1.27)) hide)
+    )
+    (property "Link" "https://www.reichelt.de/smd-widerstand-0603-10-kohm-100-mw-1--rnd-0603-1-10k-p183077.html?search=10k+0603" (id 5) (at 219.71 52.07 0)
+      (effects (font (size 1.27 1.27)) hide)
+    )
   )
   (symbol (lib_id "Device:R") (at 219.71 77.47 0) (unit 1)
@@
       (effects (font (size 1.27 1.27)) hide)
     )
+    (property "Distri" "Reichelt" (id 4) (at 219.71 77.47 0)
+      (effects (font (size 1.27 1.27)) hide)
+    )
+    (property "Link" "https://www.reichelt.de/smd-widerstand-0603-10-kohm-100-mw-1--rnd-0603-1-10k-p183077.html?search=10k+0603" (id 5) (at 219.71 77.47 0)
+      (effects (font (size 1.27 1.27)) hide)
+    )
   )
   (symbol (lib_id "Device:R") (at 219.71 102.87 0) (unit 1)
@@
       (effects (font (size 1.27 1.27)) hide)
     )
+    (property "Distri" "Reichelt" (id 4) (at 219.71 102.87 0)
+      (effects (font (size 1.27 1.27)) hide)
+    )
+    (property "Link" "https://www.reichelt.de/smd-widerstand-0603-10-kohm-100-mw-1--rnd-0603-1-10k-p183077.html?search=10k+0603" (id 5) (at 219.71 102.87 0)
+      (effects (font (size 1.27 1.27)) hide)
+    )
   )
   (symbol (lib_id "Device:R") (at 219.71 128.27 0) (unit 1)
@@
       (effects (font (size 1.27 1.27)) hide)
     )
+    (property "Distri" "Reichelt" (id 4) (at 219.71 128.27 0)
+      (effects (font (size 1.27 1.27)) hide)
+    )
+    (property "Link" "https://www.reichelt.de/smd-widerstand-0603-10-kohm-100-mw-1--rnd-0603-1-10k-p183077.html?search=10k+0603" (id 5) (at 219.71 128.27 0)
+      (effects (font (size 1.27 1.27)) hide)
+    )
   )
   (symbol (lib_id "Device:R") (at 219.71 153.67 0) (unit 1)
@@
       (effects (font (size 1.27 1.27)) hide)
     )
+    (property "Distri" "Reichelt" (id 4) (at 219.71 153.67 0)
+      (effects (font (size 1.27 1.27)) hide)
+    )
+    (property "Link" "https://www.reichelt.de/smd-widerstand-0603-10-kohm-100-mw-1--rnd-0603-1-10k-p183077.html?search=10k+0603" (id 5) (at 219.71 153.67 0)
+      (effects (font (size 1.27 1.27)) hide)
+    )
   )
   (symbol (lib_id "Device:R") (at 233.68 26.67 0) (unit 1)
@@
       (effects (font (size 1.27 1.27)) hide)
     )
+    (property "Distri" "Reichelt" (id 4) (at 233.68 26.67 0)
+      (effects (font (size 1.27 1.27)) hide)
+    )
+    (property "Link" "https://www.reichelt.de/smd-widerstand-0603-10-kohm-100-mw-1--rnd-0603-1-10k-p183077.html?search=10k+0603" (id 5) (at 233.68 26.67 0)
+      (effects (font (size 1.27 1.27)) hide)
+    )
   )
   (symbol (lib_id "Device:R") (at 233.68 52.07 0) (unit 1)
@@
       (effects (font (size 1.27 1.27)) hide)
     )
+    (property "Distri" "Reichelt" (id 4) (at 233.68 52.07 0)
+      (effects (font (size 1.27 1.27)) hide)
+    )
+    (property "Link" "https://www.reichelt.de/smd-widerstand-0603-10-kohm-100-mw-1--rnd-0603-1-10k-p183077.html?search=10k+0603" (id 5) (at 233.68 52.07 0)
+      (effects (font (size 1.27 1.27)) hide)
+    )
   )
   (symbol (lib_id "Device:R") (at 233.68 77.47 0) (unit 1)
@@
       (effects (font (size 1.27 1.27)) hide)
     )
+    (property "Distri" "Reichelt" (id 4) (at 233.68 77.47 0)
+      (effects (font (size 1.27 1.27)) hide)
+    )
+    (property "Link" "https://www.reichelt.de/smd-widerstand-0603-10-kohm-100-mw-1--rnd-0603-1-10k-p183077.html?search=10k+0603" (id 5) (at 233.68 77.47 0)
+      (effects (font (size 1.27 1.27)) hide)
+    )
   )
   (symbol (lib_id "Device:R") (at 233.68 102.87 0) (unit 1)
@@
       (effects (font (size 1.27 1.27)) hide)
     )
+    (property "Distri" "Reichelt" (id 4) (at 233.68 102.87 0)
+      (effects (font (size 1.27 1.27)) hide)
+    )
+    (property "Link" "https://www.reichelt.de/smd-widerstand-0603-10-kohm-100-mw-1--rnd-0603-1-10k-p183077.html?search=10k+0603" (id 5) (at 233.68 102.87 0)
+      (effects (font (size 1.27 1.27)) hide)
+    )
   )
   (symbol (lib_id "Device:R") (at 233.68 128.27 0) (unit 1)
@@
       (effects (font (size 1.27 1.27)) hide)
     )
+    (property "Distri" "Reichelt" (id 4) (at 233.68 128.27 0)
+      (effects (font (size 1.27 1.27)) hide)
+    )
+    (property "Link" "https://www.reichelt.de/smd-widerstand-0603-10-kohm-100-mw-1--rnd-0603-1-10k-p183077.html?search=10k+0603" (id 5) (at 233.68 128.27 0)
+      (effects (font (size 1.27 1.27)) hide)
+    )
   )
   (symbol (lib_id "Device:R") (at 233.68 153.67 0) (unit 1)
@@
       (effects (font (size 1.27 1.27)) hide)
     )
+    (property "Distri" "Reichelt" (id 4) (at 233.68 153.67 0)
+      (effects (font (size 1.27 1.27)) hide)
+    )
+    (property "Link" "https://www.reichelt.de/smd-widerstand-0603-10-kohm-100-mw-1--rnd-0603-1-10k-p183077.html?search=10k+0603" (id 5) (at 233.68 153.67 0)
+      (effects (font (size 1.27 1.27)) hide)
+    )
   )
   (symbol (lib_id "Device:R") (at 238.76 21.59 270) (unit 1)
@@
       (effects (font (size 1.27 1.27)) hide)
     )
+    (property "Distri" "Reichelt" (id 4) (at 238.76 21.59 0)
+      (effects (font (size 1.27 1.27)) hide)
+    )
+    (property "Link" "https://www.reichelt.de/smd-widerstand-0603-51-ohm-100-mw-1--rnd-0603-1-51-p183008.html?search=0603+51" (id 5) (at 238.76 21.59 0)
+      (effects (font (size 1.27 1.27)) hide)
+    )
   )
   (symbol (lib_id "Device:R") (at 238.76 46.99 270) (unit 1)
@@
       (effects (font (size 1.27 1.27)) hide)
     )
+    (property "Distri" "Reichelt" (id 4) (at 238.76 46.99 0)
+      (effects (font (size 1.27 1.27)) hide)
+    )
+    (property "Link" "https://www.reichelt.de/smd-widerstand-0603-51-ohm-100-mw-1--rnd-0603-1-51-p183008.html?search=0603+51" (id 5) (at 238.76 46.99 0)
+      (effects (font (size 1.27 1.27)) hide)
+    )
   )
   (symbol (lib_id "Device:R") (at 238.76 72.39 270) (unit 1)
@@
       (effects (font (size 1.27 1.27)) hide)
     )
+    (property "Distri" "Reichelt" (id 4) (at 238.76 72.39 0)
+      (effects (font (size 1.27 1.27)) hide)
+    )
+    (property "Link" "https://www.reichelt.de/smd-widerstand-0603-51-ohm-100-mw-1--rnd-0603-1-51-p183008.html?search=0603+51" (id 5) (at 238.76 72.39 0)
+      (effects (font (size 1.27 1.27)) hide)
+    )
   )
   (symbol (lib_id "Device:R") (at 238.76 97.79 270) (unit 1)
@@
       (effects (font (size 1.27 1.27)) hide)
     )
+    (property "Distri" "Reichelt" (id 4) (at 238.76 97.79 0)
+      (effects (font (size 1.27 1.27)) hide)
+    )
+    (property "Link" "https://www.reichelt.de/smd-widerstand-0603-51-ohm-100-mw-1--rnd-0603-1-51-p183008.html?search=0603+51" (id 5) (at 238.76 97.79 0)
+      (effects (font (size 1.27 1.27)) hide)
+    )
   )
   (symbol (lib_id "Device:R") (at 238.76 123.19 270) (unit 1)
@@
       (effects (font (size 1.27 1.27)) hide)
     )
+    (property "Distri" "Reichelt" (id 4) (at 238.76 123.19 0)
+      (effects (font (size 1.27 1.27)) hide)
+    )
+    (property "Link" "https://www.reichelt.de/smd-widerstand-0603-51-ohm-100-mw-1--rnd-0603-1-51-p183008.html?search=0603+51" (id 5) (at 238.76 123.19 0)
+      (effects (font (size 1.27 1.27)) hide)
+    )
   )
   (symbol (lib_id "Device:R") (at 238.76 148.59 270) (unit 1)
@@
       (effects (font (size 1.27 1.27)) hide)
     )
+    (property "Distri" "Reichelt" (id 4) (at 238.76 148.59 0)
+      (effects (font (size 1.27 1.27)) hide)
+    )
+    (property "Link" "https://www.reichelt.de/smd-widerstand-0603-51-ohm-100-mw-1--rnd-0603-1-51-p183008.html?search=0603+51" (id 5) (at 238.76 148.59 0)
+      (effects (font (size 1.27 1.27)) hide)
+    )
